File: bq28z610-Breakout.sch (KiCad schematic (older format))
At the start: 29 parts

Commit message: finished schematics
Parts:
- removed C?: 100nF, symbol C
- removed P?: CONN_01X04, symbol CONN_01X04
- removed P?: CONN_01X02, symbol CONN_01X02
- removed Q? (x2): Q_NMOS_DGS, symbol Q_NMOS_DGS
- added C10, C7, C9: 100nF, Capacitors_SMD:C_0805, symbol C
- added C6: 1µF, Capacitors_SMD:C_0805, symbol C
- added F1: Fuse, TO_SOT_Packages_SMD:SOT-23, symbol Fuse
- added P1: CONN_01X05, Pin_Headers:Pin_Header_Straight_1x05_Pitch2.54mm, symbol CONN_01X05
- added Q1, Q2: CSD16412Q5A, TO_SOT_Packages_SMD:TDSON-8-1, symbol CSD16412Q5A
- C1, C2, C3, C4, C5, C8: renamed from C?; footprint (none) -> Capacitors_SMD:C_0805
- D1: renamed from D?; footprint (none) -> TO_SOT_Packages_SMD:SOT-23
- P2, P5: renamed from P?; footprint (none) -> Pin_Headers:Pin_Header_Straight_1x02_Pitch2.54mm
- P3: renamed from P?; footprint (none) -> Connectors_JST:JST_PH_B2B-PH-SM4-TB_02x2.00mm_Straight
- P4: renamed from P?; footprint (none) -> Connectors_JST:JST_XH_B04B-XH-A_04x2.50mm_Straight
- R1, R10, R11, R12, R2, R3, R5, R6, R7, R8, R9: renamed from R?; footprint (none) -> Resistors_SMD:R_0805
- R4: renamed from R?; value ?mΩ -> 2mΩ
- gave numbers to parts that had none: 1
Connections:
- net +BATT: now also R9.2, C9.2, P1.5 (P5), Q1.1 (S), Q1.2 (S), Q1.3 (S); no longer R9.1
- net GND: now also C4.2, P5.2 (P2), R4.1, R5.1, C7.1; no longer C4.1
- net GNDPWR: now also C10.1, P1.1 (P1)
- net TS: now also P1.4 (P4)
- net at U1.10 (PBI): now also C4.1; no longer C4.2
- net VC2: now reaches U1.11 (VC2)
- net VC2: now also R10.2, C6.2
- net VC1: now reaches U1.12 (VC1)
- net VC1: now also R11.2, C6.1, C7.2
- net SDA: now reaches R2.1
- net SDA: now also P1.2 (P2)
- net SCL: now reaches R1.1
- net SCL: now also P1.3 (P3)
- net at P5.1 (P1): now also P4.1 (P1), F1.2
- net at C8.1, R12.2: now also F1.1, Q2.1 (S), Q2.2 (S), Q2.3 (S); no longer P4.1 (P1)
- net at R12.1, R7.1: now also Q2.4 (G)
- net at R8.1: now also R9.1, Q1.4 (G); no longer R9.2
- new net: Q1.5 (D), Q1.6 (D), Q1.7 (D), Q1.8 (D), Q2.5 (D), Q2.6 (D), Q2.7 (D), Q2.8 (D)
- new net: C10.2, C9.1
Other:
- moved on the sheet: C1, C2, C3, C4, C5, C8, D1, P2, P3, P4, P5, R1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

Commit message: update pictures
Parts:
- F1: footprint TO_SOT_Packages_SMD:SOT-23 -> Fuse_Holders_and_Fuses:Fuse_SMD1206_Wave
- R4: footprint (none) -> Resistors_SMD:R_2512
- U1: footprint (none) -> smd_ic:PDSO-N12
Changed lines of the file:
@@
 F 0 "U1" H 4600 3350 60  0000 C CNN
 F 1 "bq28z610" H 4450 4150 60  0000 C CNN
-F 2 "" H 4450 3750 60  0001 C CNN
+F 2 "smd_ic:PDSO-N12" H 4450 3750 60  0001 C CNN
 F 3 "" H 4450 3750 60  0001 C CNN
 	1    4450 3750
@@
 F 0 "R4" V 3230 4850 50  0000 C CNN
 F 1 "2mΩ" V 3150 4850 50  0000 C CNN
-F 2 "" V 3080 4850 50  0001 C CNN
+F 2 "Resistors_SMD:R_2512" V 3080 4850 50  0001 C CNN
 F 3 "" H 3150 4850 50  0000 C CNN
 	1    3150 4850
@@
 F 0 "F1" V 8680 3350 50  0000 C CNN
 F 1 "Fuse" V 8525 3350 50  0000 C CNN
-F 2 "TO_SOT_Packages_SMD:SOT-23" V 8530 3350 50  0001 C CNN
+F 2 "Fuse_Holders_and_Fuses:Fuse_SMD1206_Wave" V 8530 3350 50  0001 C CNN
 F 3 "" H 8600 3350 50  0000 C CNN
 	1    8600 3350
